File: SensorFeatherWing/hardware/250100020129x-HW-V2.2.brd (EAGLE design)
At the start: 50.8 x 22.9 mm, 41 parts, among them CON1 n.m., CON2 QWIIC_RIGHT_ANGLE, CON3 QWIIC_RIGHT_ANGLE, CON4 2x3, CON5 2x3, IC1 2511020213301, IC2 2533020201601, IC3 2521020222501, IC4 2523020210001

Commit message: Bug fix + documentation update
Parts:
- IC4: value 2523020210001 -> 2525020210001; device WSen-HIDS:WSEN-HIDS_0202 -> WE_WSEN-Rev4.1:WSEN-HIDS_2525020210001
Changed lines of the file:
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@@
 <?xml version="1.0" encoding="utf-8"?>
 <!DOCTYPE eagle SYSTEM "eagle.dtd">
-<eagle version="7.5.0">
+<eagle version="7.7.0">
 <drawing>
 <settings>
@@
 <layer number="29" name="tStop" color="7" fill="3" visible="no" active="yes"/>
 <layer number="30" name="bStop" color="7" fill="6" visible="no" active="yes"/>
-<layer number="31" name="tCream" color="7" fill="4" visible="yes" active="yes"/>
+<layer number="31" name="tCream" color="7" fill="4" visible="no" active="yes"/>
 <layer number="32" name="bCream" color="7" fill="5" visible="no" active="yes"/>
 <layer number="33" name="tFinish" color="6" fill="3" visible="no" active="yes"/>
@@
 <layer number="49" name="Reference" color="7" fill="1" visible="no" active="yes"/>
 <layer number="50" name="dxf" color="7" fill="1" visible="no" active="no"/>
-<layer number="51" name="tDocu" color="7" fill="1" visible="yes" active="yes"/>
+<layer number="51" name="tDocu" color="7" fill="1" visible="no" active="yes"/>
 <layer number="52" name="bDocu" color="7" fill="1" visible="no" active="yes"/>
 <layer number="53" name="tGND_GNDA" color="7" fill="9" visible="no" active="no"/>
@@
 <attribute name="VALUE" x="22.35" y="17" size="0.4064" layer="27"/>
 </element>
-<element name="IC4" library="WSen-HIDS" package="WSEN-HIDS_0202" value="2523020210001" x="36" y="11.5" smashed="yes" rot="R180">
+<element name="IC4" library="WE_WSEN-Rev4.1" package="WSEN-HIDS_2525020210001" value="2525020210001" x="36" y="11.5" smashed="yes" rot="R180">
 <attribute name="HEIGHT" value="1.0mm" x="38.6" y="7.15" size="1.778" layer="27" rot="R180" display="off"/>
-<attribute name="NR" value="2523020210001" x="38.6" y="7.15" size="1.778" layer="27" rot="R180" display="off"/>
-<attribute name="MANUFACTURER" value="Wurth Elektronik" x="38.6" y="7.15" size="1.778" layer="27" rot="R180" display="off"/>
+<attribute name="NR" value="2525020210001" x="38.6" y="7.15" size="1.778" layer="27" rot="R180" display="off"/>
+<attribute name="MANUFACTURER" value="Würth Elektronik" x="38.6" y="7.15" size="1.778" layer="27" rot="R180" display="off"/>
 <attribute name="PACK" value="SMD" x="38.6" y="7.15" size="1.778" layer="27" rot="R180" display="off"/>
 <attribute name="NAME" x="38.55" y="9.55" size="0.8128" layer="25" font="vector" rot="R180"/>
