File: SensorFeatherWing/hardware/250100020129x-HW-V2.2.sch (EAGLE design)
At the start: 33 parts, among them CON1 n.m., CON2 QWIIC_RIGHT_ANGLE, CON3 QWIIC_RIGHT_ANGLE, CON4 2x3, CON5 2x3, IC1 2511020213301, IC2 2533020201601, IC3 2521020222501, IC4 2523020210001

Commit message: Bug fix + documentation update
Parts:
- IC4: value 2523020210001 -> 2525020210001; device WSen-HIDS:WSEN-HIDS -> WE_WSEN-Rev4.1:WSEN-HIDS_2525020210001; MANUFACTURER Wurth Elektronik -> (none); NR 2523020210001 -> (none)
Connections:
- net DRDY_HIDS: now also IC4.INT; no longer IC4.DRDY
Changed lines of the file:
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@@
 <?xml version="1.0" encoding="utf-8"?>
 <!DOCTYPE eagle SYSTEM "eagle.dtd">
-<eagle version="7.5.0">
+<eagle version="7.7.0">
 <drawing>
 <settings>
@@
 <part name="R10" library="rcl-amber" deviceset="R" device="0402_IPC" technology="0R" value="0R"/>
 <part name="R11" library="rcl-amber" deviceset="R" device="0402_IPC" value="n.m."/>
-<part name="IC4" library="WSen-HIDS" deviceset="WSEN-HIDS" device="" value="2523020210001">
+<part name="IC4" library="WE_WSEN-Rev4.1" deviceset="WSEN-HIDS_2525020210001" device="" value="2525020210001">
 <attribute name="HEIGHT" value="1.0mm"/>
-<attribute name="MANUFACTURER" value="Wurth Elektronik"/>
-<attribute name="NR" value="2523020210001"/>
 <attribute name="PACK" value="SMD"/>
 </part>
@@
 <net name="DRDY_HIDS" class="0">
 <segment>
-<pinref part="IC4" gate="G$1" pin="DRDY"/>
+<pinref part="IC4" gate="G$1" pin="INT"/>
 <wire x1="170.18" y1="43.18" x2="165.1" y2="43.18" width="0.1524" layer="91"/>
 <label x="165.1" y="43.18" size="1.4224" layer="95" rot="R180" xref="yes"/>
