File: SensorFeatherWing/hardware/250100020129x-HW-V2.4.brd (EAGLE design)
At the start: 50.8 x 22.9 mm, 41 parts, among them CON1 n.m., CON2 QWIIC_RIGHT_ANGLE, CON3 QWIIC_RIGHT_ANGLE, CON4 2x3, CON5 2x3, IC1 2511020213301, IC2 2533020201601, IC3 2521020222501, IC4 2525020210001

Commit message: Updated hardware design files
Parts:
- C10, C11, C12, C3, C4, C5, C6, C7, C8, C9: device rcl-amber:C0402_IPC -> rcl-WE:C0402_IPC
Other:
- board text added: "ACHTUNG: IC1, IC2, IC3, IC4 sind empfindliche Komponenten. Die Pastendaten dürfen in der absoluten Ausdehnung nicht verändert werden."
- board text added: "JP1: GPIOA5 - SPI_CE"
- board text removed: "JP1: GPIOA4 - INT"
