File: SensorFeatherWing/hardware/250100020129x-HW-V2.4.sch (EAGLE design)
At the start: 33 parts, among them CON1 n.m., CON2 QWIIC_RIGHT_ANGLE, CON3 QWIIC_RIGHT_ANGLE, CON4 2x3, CON5 2x3, IC1 2511020213301, IC2 2533020201601, IC3 2521020222501, IC4 2525020210001

Commit message: Updated hardware design files
Parts:
- C10, C12, C4, C6, C7, C9: device rcl-amber:C100NF0402_IPC -> rcl-WE:C100NF0402_IPC
- C11, C5, C8: device rcl-amber:C10UF0402_IPC -> rcl-WE:C10UF0402_IPC
- C3: device rcl-amber:C4,7UF0402_IPC -> rcl-WE:C4.7UF0402_IPC
