File: CalypsoWiFiFeatherWing/hardware/261003902xxxx-HW-V1.3.sch (EAGLE design)
At the start: 32 parts, among them T1 BSS138, T2 BSS138

Commit message: Updated hardware design files
Parts:
- C4: device rcl-amber:C22PF0402_IPC -> rcl-WE:C22PF0402_IPC
- C6: device rcl-amber:C100NF0402_IPC -> rcl-WE:C100NF0402_IPC
- C7: device rcl-amber:C1UF0402_IPC -> rcl-WE:C1UF0402_IPC
Connections:
- net APP_MODE_0: now also JP2.4, JP3.5, MOD1.10; no longer JP2.3, JP3.3, MOD1.11
- net APP_MODE_1: now also JP2.3, JP3.3, MOD1.11; no longer JP2.4, JP3.5, MOD1.10
Changed lines of the file:
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@@
 <?xml version="1.0" encoding="utf-8"?>
 <!DOCTYPE eagle SYSTEM "eagle.dtd">
-<eagle version="7.5.0">
+<eagle version="7.7.0">
 <drawing>
 <settings>
@@
 <part name="C2" library="rcl-amber" deviceset="C" device="0201_IPC" value="n.m."/>
 <part name="C3" library="rcl-amber" deviceset="C" device="0201_IPC" value="n.m."/>
-<part name="C4" library="rcl-amber" deviceset="C" device="0402_IPC" technology="22PF" value="22pF"/>
+<part name="C4" library="rcl-WE" deviceset="C" device="0402_IPC" technology="22PF" value="22pF"/>
 <part name="GND3" library="supply1" deviceset="GND" device=""/>
 <part name="GND4" library="supply1" deviceset="GND" device=""/>
@@
 <part name="GND7" library="supply1" deviceset="GND" device=""/>
 <part name="C5" library="rcl-WE" deviceset="C" device="0402_IPC" technology="4.7UF" value="4u7"/>
-<part name="C6" library="rcl-amber" deviceset="C" device="0402_IPC" technology="100NF" value="100nF"/>
+<part name="C6" library="rcl-WE" deviceset="C" device="0402_IPC" technology="100NF" value="100nF"/>
 <part name="GND8" library="supply1" deviceset="GND" device=""/>
 <part name="GND9" library="supply1" deviceset="GND" device=""/>
@@
 <part name="+3V10" library="supply1" deviceset="+3V3" device=""/>
 <part name="R6" library="rcl-amber" deviceset="R" device="0402_IPC" technology="10KR" value="10kR"/>
-<part name="C7" library="rcl-amber" deviceset="C" device="0402_IPC" technology="1UF" value="1uF"/>
+<part name="C7" library="rcl-WE" deviceset="C" device="0402_IPC" technology="1UF" value="1uF"/>
 <part name="GND15" library="supply1" deviceset="GND" device=""/>
 <part name="TP1" library="testpad" deviceset="TP-DRILL" device="0.6" value="n.m."/>
@@
 </segment>
 </net>
-<net name="APP_MODE_1" class="0">
+<net name="APP_MODE_0" class="0">
 <segment>
 <pinref part="MOD1" gate="G$1" pin="10"/>
@@
 </segment>
 </net>
-<net name="APP_MODE_0" class="0">
+<net name="APP_MODE_1" class="0">
 <segment>
 <pinref part="MOD1" gate="G$1" pin="11"/>
