File: ThyoneWirelessFeatherWing/hardware/261105902xxxx-HW-V2.1.sch (EAGLE design)
At the start: 46 parts, among them CON1 1x2, CON2 n.m., IC1 ATECC608A, Q3 32.768kHz, T1 MOSFET-NCH-BSS138, T2 MOSFET-NCH-BSS138

Commit message: Updated hardware design files
Parts:
- removed CON1, JP3: 1x2, pinhead:PINHD-1X2/R
- removed JP1: 2x3, pinhead:PINHD-2X3
- added SJ1, SJ2, SJ4, SJ5, SJ6: (no value), jumper:SJ
- added SJ3: (no value), jumper:SJ_SHUNTD
- added TP1, TP2: TP15R, testpad:TP15R
- IC1: value ATECC608A -> ATECC608B; device wuerth_io:ATECC608ASOIC8 -> microchip:ATECC608B-TNGTLS; HEIGHT 1.75mm -> (none); NR ATECC608A-TNGTLSS-C -> (none); PACK SOIC-8 -> UDFN-8
- Q3: MANUFACTURER (none) -> Würth Elektronik; MANUFACTURER2 IQD -> (none); MANUFACTURER_2 (none) -> Microcrystal; NR CM7V-T1A-32.768k-9pF-20PPM-TA-QA T3 -> 830009706; NR2 LFXTAL009706Reel -> (none); NR_2 (none) -> CM7V-T1A-32.768k-9pF-20PPM-TA-QA T3
- R1: value 4kR -> 4k7R
Connections:
- new net /CTS: MOD1.P0.12/!CTS, SJ6.2
- new net /RTS: MOD1.P0.11/!RTS, SJ5.2
- new net N$13: MS1.GPIO6, SJ5.1
- new net N$14: MS1.GPIO5, SJ6.1
- new net RESERVED1: MS1.GPIOA0, SJ4.1
- new net SWDCLK: MOD1.SWDCLK, TP1.TP
- new net SWDIO: MOD1.SWDIO, TP2.TP
- net GND: no longer CON1.1
- net GPIO13: now also SJ3.1; no longer JP1.5
- net GPIO9: now also SJ1.1; no longer JP1.1
- net GPIOA3: now also SJ2.1; no longer JP1.3
- net N$8: now also MOD1.B1, SJ4.2; no longer CON1.2, JP3.2
- net OP_MODE: now also SJ2.2; no longer JP1.4
- net S2: now also SJ3.2; no longer JP1.6
- net VCC: no longer JP3.1
- net WAKE_UP: now also SJ1.2; no longer JP1.2
Other:
- moved on the sheet: C7, IC1, O1, O2
